File: esp32-lifepo4.sch (KiCad schematic (older format))
At the start: 14 parts, among them J1 Conn_01x12, J2 Conn_01x12, U1 ESP32-WROOM-32, U2 CN3058C, U3 TPS709

Commit message: v0
Parts:
- removed D1: DIODE, Diodes_SMD:D_SMA, symbol pspice:DIODE
- C1: LCSC (none) -> C28323
- C2: value 4.7-10uF -> 10uF; LCSC (none) -> C15850
- D2: value LED -> DONE; LCSC (none) -> C2286
- D3: value LED -> CHRG; LCSC (none) -> C2286
- J1, J2, JP1, U3: ignorebom (none) -> 1
- R1: value 100 -> 100 ohms; LCSC (none) -> C17408
- R2: value 2.463k -> 2.463k ohms; LCSC (none) -> C17526
- R3: value 0 -> 0ohm; LCSC (none) -> C17477
- U1: LCSC (none) -> C95209
- U2: value CN3058C -> CN3058E; LCSC (none) -> C112011
Connections:
- net VIN: now also C1.2, R1.2, U2.4 (VIN)
Changed lines of the file:
@@
 EESchema Schematic File Version 4
+LIBS:esp32-lifepo4-cache
 EELAYER 26 0
 EELAYER END
@@
 P 5050 2100
 F 0 "U2" H 5218 2565 50  0000 C CNN
-F 1 "CN3058C" H 5218 2474 50  0000 C CNN
+F 1 "CN3058E" H 5218 2474 50  0000 C CNN
 F 2 "Housings_SOIC:SOIC-8_3.9x4.9mm_Pitch1.27mm" H 5250 2450 50  0001 C CNN
 F 3 "" H 5250 2450 50  0001 C CNN
+F 4 "C112011" H 0   0   50  0001 C CNN "LCSC"
 	1    5050 2100
 	1    0    0    -1
@@
 P 6200 2050
 F 0 "R3" V 6100 2150 50  0000 C CNN
-F 1 "0" V 6100 2000 50  0000 C CNN
+F 1 "0ohm" V 6100 2000 50  0000 C CNN
 F 2 "Resistors:0805" V 6130 2050 50  0001 C CNN
 F 3 "~" H 6200 2050 50  0001 C CNN
+F 4 "C17477" H 0   0   50  0001 C CNN "LCSC"
 	1    6200 2050
 	0    1    1    0
@@
 P 5700 2650
 F 0 "R2" H 5630 2604 50  0000 R CNN
-F 1 "2.463k" H 5630 2695 50  0000 R CNN
+F 1 "2.463k ohms" H 5630 2695 50  0000 R CNN
 F 2 "Resistors:0805" V 5630 2650 50  0001 C CNN
 F 3 "~" H 5700 2650 50  0001 C CNN
+F 4 "C17526" H 5700 2650 50  0001 C CNN "LCSC"
 	1    5700 2650
 	-1   0    0    1
@@
 P 3750 2050
 F 0 "R1" H 3680 2004 50  0000 R CNN
-F 1 "100" H 3680 2095 50  0000 R CNN
+F 1 "100 ohms" V 3850 2300 50  0000 R CNN
 F 2 "Resistors:0805" V 3680 2050 50  0001 C CNN
 F 3 "~" H 3750 2050 50  0001 C CNN
+F 4 "C17408" H 0   0   50  0001 C CNN "LCSC"
 	1    3750 2050
 	-1   0    0    1
@@
 P 5800 1750
 F 0 "C2" H 5915 1796 50  0000 L CNN
-F 1 "4.7-10uF" H 5915 1705 50  0000 L CNN
+F 1 "10uF" H 5915 1705 50  0000 L CNN
 F 2 "Capacitors_SMD:C_0805" H 5838 1600 50  0001 C CNN
 F 3 "~" H 5800 1750 50  0001 C CNN
+F 4 "C15850" H 0   0   50  0001 C CNN "LCSC"
 	1    5800 1750
 	1    0    0    -1
@@
 F 2 "Capacitors_SMD:C_0805" H 4338 1600 50  0001 C CNN
 F 3 "~" H 4300 1750 50  0001 C CNN
+F 4 "C28323" H 0   0   50  0001 C CNN "LCSC"
 	1    4300 1750
 	1    0    0    -1
@@
 	-1   0    0    1
 $EndComp
-$Comp
-L pspice:DIODE D1
-U 1 1 5D9D1436
-P 3000 1900
-F 0 "D1" H 3000 2165 50  0000 C CNN
-F 1 "DIODE" H 3000 2074 50  0000 C CNN
-F 2 "Diodes_SMD:D_SMA" H 3000 1900 50  0001 C CNN
-F 3 "~" H 3000 1900 50  0001 C CNN
-	1    3000 1900
-	1    0    0    -1
-$EndComp
-Wire Wire Line
-	3200 1900 3750 1900
 Connection ~ 3750 1900
 Wire Wire Line
@@
 P 4200 2200
 F 0 "D2" H 4350 2100 50  0000 C CNN
-F 1 "LED" H 4200 2100 50  0000 C CNN
+F 1 "DONE" H 4150 2100 50  0000 C CNN
 F 2 "LEDs:LED_0603" H 4200 2200 50  0001 C CNN
 F 3 "~" H 4200 2200 50  0001 C CNN
+F 4 "C2286" H 0   0   50  0001 C CNN "LCSC"
 	1    4200 2200
 	-1   0    0    1
@@
 U 1 1 5D9D1926
 P 4200 2350
-F 0 "D3" H 4300 2450 50  0000 C CNN
-F 1 "LED" H 4150 2450 50  0000 C CNN
+F 0 "D3" H 4350 2450 50  0000 C CNN
+F 1 "CHRG" H 4150 2450 50  0000 C CNN
 F 2 "LEDs:LED_0603" H 4200 2350 50  0001 C CNN
 F 3 "~" H 4200 2350 50  0001 C CNN
+F 4 "C2286" H 0   0   50  0001 C CNN "LCSC"
 	1    4200 2350
 	-1   0    0    1
@@
 	1    0    0    -1
 $EndComp
-Text GLabel 2550 1900 0    50   Input ~ 0
+Text GLabel 3150 1900 0    50   Input ~ 0
 VIN
 Text GLabel 10200 1900 2    50   Input ~ 0
@@
 F 2 "TO_SOT_Packages_SMD:SOT-23-5" H 8250 1650 50  0001 C CNN
 F 3 "" H 8250 1650 50  0001 C CNN
+F 4 "1" H 8800 2000 50  0001 C CNN "ignorebom"
 	1    8800 2000
 	1    0    0    -1
@@
 F 2 "Jumpers:SMT-JUMPER_2_NO_SILK" H 8800 1250 50  0001 C CNN
 F 3 "~" H 8800 1250 50  0001 C CNN
+F 4 "" H 8800 1250 50  0001 C CNN "nobom"
+F 5 "1" H 0   0   50  0001 C CNN "ignorebom"
 	1    8800 1250
 	1    0    0    -1
@@
 F 2 "symbols:ESP32-WROOM-32-Espressif-Symbol-Kicad-62379" H 3250 5100 60  0001 C CNN
 F 3 "" H 3250 5100 60  0001 C CNN
+F 4 "C95209" H 0   0   50  0001 C CNN "LCSC"
 	1    3200 5200
 	1    0    0    -1
@@
 F 2 "Connectors Sparkfun:1X12" H 6650 5150 50  0001 C CNN
 F 3 "~" H 6650 5150 50  0001 C CNN
+F 4 "" H 6650 5150 50  0001 C CNN "nobom"
+F 5 "1" H 0   0   50  0001 C CNN "ignorebom"
 	1    6650 5150
 	1    0    0    -1
@@
 F 2 "Connectors Sparkfun:1X12" H 7750 5250 50  0001 C CNN
 F 3 "~" H 7750 5250 50  0001 C CNN
+F 4 "" H 7750 5250 50  0001 C CNN "nobom"
+F 5 "1" H 0   0   50  0001 C CNN "ignorebom"
 	1    7750 5250
 	-1   0    0    1
@@
 	2600 6550 2600 6650
 Connection ~ 2600 6550
-Wire Wire Line
-	2550 1900 2800 1900
 $Comp
 L power:PWR_FLAG #FLG0101
@@
 Wire Wire Line
 	2600 6650 2600 6750
+Wire Wire Line
+	3150 1900 3750 1900
 $EndSCHEMATC
